Commit message: modified example

File: resources/ffw_sg2/ffw_sg2_planning.urdf (robot description, URDF)
Before this commit: robot ffw_sg2_follower, 40 links, 39 joints
Links:
- removed link camera_l_bottom_screw_frame
- removed link camera_l_link
- removed link camera_r_bottom_screw_frame
- removed link camera_r_link
- removed link world
- added link camera_left_bottom_screw_frame
- added link camera_left_link; collision box size=0.023 0.042 0.042
- added link camera_right_bottom_screw_frame
- added link camera_right_link; collision box size=0.023 0.042 0.042
- added link end_effector_l_link
- added link end_effector_r_link
- added link imu_link
- added link lidar_l_link
- added link lidar_r_link
- added link zed_camera_center; collision mesh filename=../../ai_worker/ffw_description/meshes/common/follower/zedm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 scale=0.001 0.001 0.001
- added link zed_camera_link
- added link zed_left_camera_frame
- added link zed_left_camera_optical_frame
- added link zed_right_camera_frame
- added link zed_right_camera_optical_frame
- link arm_base_link: geometry collision mesh filename=../../ai_worker/ffw_description/meshes/common/follower/ffw/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 scale=0.001 0.001 0.001
- link arm_l_link1: geometry collision mesh filename=../../ai_worker/ffw_description/meshes/common/follower/ffw/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 scale=0.001 0.001 0.001
- link arm_l_link2: geometry collision mesh filename=../../ai_worker/ffw_description/meshes/common/follower/ffw/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 scale=0.001 0.001 0.001
- link arm_l_link3: geometry collision mesh filename=../../ai_worker/ffw_description/meshes/common/follower/ffw/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 scale=0.001 0.001 0.001
- link arm_l_link4: geometry collision mesh filename=../../ai_worker/ffw_description/meshes/common/follower/ffw/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 scale=0.001 0.001 0.001
- link arm_l_link5: geometry collision mesh filename=../../ai_worker/ffw_description/meshes/common/follower/ffw/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 scale=0.001 0.001 0.001
- link arm_l_link6: geometry collision mesh filename=../../ai_worker/ffw_description/meshes/common/follower/ffw/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 scale=0.001 0.001 0.001
- link arm_l_link7: geometry collision mesh filename=../../ai_worker/ffw_description/meshes/common/follower/ffw/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 scale=0.001 0.001 0.001
- link arm_r_link1: geometry collision mesh filename=../../ai_worker/ffw_description/meshes/common/follower/ffw/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 scale=0.001 0.001 0.001
- link arm_r_link2: geometry collision mesh filename=../../ai_worker/ffw_description/meshes/common/follower/ffw/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 scale=0.001 0.001 0.001
- link arm_r_link3: geometry collision mesh filename=../../ai_worker/ffw_description/meshes/common/follower/ffw/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 scale=0.001 0.001 0.001
- link arm_r_link4: geometry collision mesh filename=../../ai_worker/ffw_description/meshes/common/follower/ffw/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 scale=0.001 0.001 0.001
- link arm_r_link5: geometry collision mesh filename=../../ai_worker/ffw_description/meshes/common/follower/ffw/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 scale=0.001 0.001 0.001
- link arm_r_link6: geometry collision mesh filename=../../ai_worker/ffw_description/meshes/common/follower/ffw/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 scale=0.001 0.001 0.001
- link arm_r_link7: geometry collision mesh filename=../../ai_worker/ffw_description/meshes/common/follower/ffw/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 scale=0.001 0.001 0.001
- link base_link: geometry collision mesh filename=../../ai_worker/ffw_description/meshes/common/follower/ffw_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 scale=0.001 0.001 0.001
- link gripper_l_rh_p12_rn_base: geometry collision mesh filename=../../ai_worker/ffw_description/meshes/common/rh_p12_rn_a/b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 scale=0.001 0.001 0.001
- link gripper_l_rh_p12_rn_l1: geometry collision mesh filename=../../ai_worker/ffw_description/meshes/common/rh_p12_rn_a/l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 scale=0.001 0.001 0.001
- link gripper_l_rh_p12_rn_l2: geometry collision mesh filename=../../ai_worker/ffw_description/meshes/common/rh_p12_rn_a/l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 scale=0.001 0.001 0.001
- link gripper_l_rh_p12_rn_r1: geometry collision mesh filename=../../ai_worker/ffw_description/meshes/common/rh_p12_rn_a/r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 scale=0.001 0.001 0.001
- link gripper_l_rh_p12_rn_r2: geometry collision mesh filename=../../ai_worker/ffw_description/meshes/common/rh_p12_rn_a/r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 scale=0.001 0.001 0.001
- link gripper_r_rh_p12_rn_base: geometry collision mesh filename=../../ai_worker/ffw_description/meshes/common/rh_p12_rn_a/b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 scale=0.001 0.001 0.001
- link gripper_r_rh_p12_rn_l1: geometry collision mesh filename=../../ai_worker/ffw_description/meshes/common/rh_p12_rn_a/l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 scale=0.001 0.001 0.001
- link gripper_r_rh_p12_rn_l2: geometry collision mesh filename=../../ai_worker/ffw_description/meshes/common/rh_p12_rn_a/l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 scale=0.001 0.001 0.001
- link gripper_r_rh_p12_rn_r1: geometry collision mesh filename=../../ai_worker/ffw_description/meshes/common/rh_p12_rn_a/r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 scale=0.001 0.001 0.001
- link gripper_r_rh_p12_rn_r2: geometry collision mesh filename=../../ai_worker/ffw_description/meshes/common/rh_p12_rn_a/r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 scale=0.001 0.001 0.001
- link head_link1: geometry collision mesh filename=../../ai_worker/ffw_description/meshes/common/follower/ffw/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 scale=0.001 0.001 0.001
- link head_link2: geometry collision mesh filename=../../ai_worker/ffw_description/meshes/common/follower/ffw/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 scale=0.001 0.001 0.001
- link left_wheel_drive_link: geometry collision cylinder length=0.05 radius=0.0865
- link left_wheel_steer_link: geometry collision mesh filename=../../ai_worker/ffw_description/meshes/common/follower/ffw_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 scale=0.001 0.001 0.001
- link lift_link: geometry collision mesh filename=../../ai_worker/ffw_description/meshes/common/follower/ffw_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 scale=0.001 0.001 0.001
- link rear_wheel_drive_link: geometry collision cylinder length=0.05 radius=0.0865
- link rear_wheel_steer_link: geometry collision mesh filename=../../ai_worker/ffw_description/meshes/common/follower/ffw_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 scale=0.001 0.001 0.001
- link right_wheel_drive_link: geometry collision cylinder length=0.05 radius=0.0865
- link right_wheel_steer_link: geometry collision mesh filename=../../ai_worker/ffw_description/meshes/common/follower/ffw_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 scale=0.001 0.001 0.001
Joints:
- removed joint camera_l_joint
- removed joint camera_l_link_joint
- removed joint camera_r_joint
- removed joint camera_r_link_joint
- removed joint world_fixed
- added joint camera_left_joint: type fixed, parent arm_l_link7, child camera_left_bottom_screw_frame, origin xyz=0.108236 -0.021 -0.062552 rpy=-1.57079632679 1.66678943569 0
- added joint camera_left_link_joint: type fixed, parent camera_left_bottom_screw_frame, child camera_left_link, origin xyz=0.01085 0.009 0.021 rpy=0 0 0
- added joint camera_right_joint: type fixed, parent arm_r_link7, child camera_right_bottom_screw_frame, origin xyz=0.108236 -0.021 -0.062552 rpy=-1.57079632679 1.66678943569 0
- added joint camera_right_link_joint: type fixed, parent camera_right_bottom_screw_frame, child camera_right_link, origin xyz=0.01085 0.009 0.021 rpy=0 0 0
- added joint end_effector_l_joint: type fixed, parent arm_l_link7, child end_effector_l_link, origin xyz=0 0 -0.215 rpy=0 0 0
- added joint end_effector_r_joint: type fixed, parent arm_r_link7, child end_effector_r_link, origin xyz=0 0 -0.215 rpy=0 0 0
- added joint imu_joint: type fixed, parent base_link, child imu_link, origin xyz=-0.1464 0.0 0.26 rpy=0 0 0
- added joint lidar_l_joint: type fixed, parent base_link, child lidar_l_link, origin xyz=-0.111881 0.240 0.34432 rpy=0 0 1.57079632679
- added joint lidar_r_joint: type fixed, parent base_link, child lidar_r_link, origin xyz=-0.111881 -0.240 0.34432 rpy=0 0 -1.57079632679
- added joint zed_camera_center_joint: type fixed, parent zed_camera_link, child zed_camera_center, origin xyz=0 0 0.01325 rpy=0 0 0
- added joint zed_joint: type fixed, parent head_link2, child zed_camera_link, origin xyz=0.0238122 -0.00651797 -0.0242094 rpy=0 0 0
- added joint zed_left_camera_joint: type fixed, parent zed_camera_center, child zed_left_camera_frame, origin xyz=0 0.0315 0 rpy=0 0 0
- added joint zed_left_camera_optical_joint: type fixed, parent zed_left_camera_frame, child zed_left_camera_optical_frame, origin xyz=0 0 0 rpy=-1.57079632679 0.0 -1.57079632679
- added joint zed_right_camera_joint: type fixed, parent zed_camera_center, child zed_right_camera_frame, origin xyz=0 -0.0315 0 rpy=0 0 0
- added joint zed_right_camera_optical_joint: type fixed, parent zed_right_camera_frame, child zed_right_camera_optical_frame, origin xyz=0 0 0 rpy=-1.57079632679 0.0 -1.57079632679
- joint arm_l_joint7: limit lower=-1.8201 upper=1.5804 effort=1000 velocity=4.8 -> lower=-1.5804 upper=1.8201 effort=1000 velocity=4.8
- joint arm_r_joint7: limit lower=-1.5804 upper=1.8201 effort=1000 velocity=4.8 -> lower=-1.8201 upper=1.5804 effort=1000 velocity=4.8
- joint head_joint1: origin xyz=0.0494878 0 0.102123 rpy=0 0 0 -> xyz=0.049483 0 0.102130 rpy=0 0 0
- joint head_joint2: origin xyz=0.0365694 0 0.0563797 rpy=0 0 0 -> xyz=0.040 0 0.054 rpy=0 0 0

File: resources/ffw_sg2/ffw_sg2_spherized.urdf (robot description, URDF)
Before this commit: robot ffw_sg2_follower, 40 links, 39 joints
Links:
- removed link camera_l_bottom_screw_frame
- removed link camera_l_link
- removed link camera_r_bottom_screw_frame
- removed link camera_r_link
- removed link world
- added link camera_left_bottom_screw_frame
- added link camera_left_link
- added link camera_right_bottom_screw_frame
- added link camera_right_link
- added link end_effector_l_link
- added link end_effector_r_link
- added link imu_link
- added link lidar_l_link
- added link lidar_r_link
- added link zed_camera_center
- added link zed_camera_link
- added link zed_left_camera_frame
- added link zed_left_camera_optical_frame
- added link zed_right_camera_frame
- added link zed_right_camera_optical_frame
Joints:
- removed joint camera_l_joint
- removed joint camera_l_link_joint
- removed joint camera_r_joint
- removed joint camera_r_link_joint
- removed joint world_fixed
- added joint camera_left_joint: type fixed, parent arm_l_link7, child camera_left_bottom_screw_frame, origin xyz=0.108236 -0.021 -0.062552 rpy=-1.57079632679 1.66678943569 0
- added joint camera_left_link_joint: type fixed, parent camera_left_bottom_screw_frame, child camera_left_link, origin xyz=0.01085 0.009 0.021 rpy=0 0 0
- added joint camera_right_joint: type fixed, parent arm_r_link7, child camera_right_bottom_screw_frame, origin xyz=0.108236 -0.021 -0.062552 rpy=-1.57079632679 1.66678943569 0
- added joint camera_right_link_joint: type fixed, parent camera_right_bottom_screw_frame, child camera_right_link, origin xyz=0.01085 0.009 0.021 rpy=0 0 0
- added joint end_effector_l_joint: type fixed, parent arm_l_link7, child end_effector_l_link, origin xyz=0 0 -0.215 rpy=0 0 0
- added joint end_effector_r_joint: type fixed, parent arm_r_link7, child end_effector_r_link, origin xyz=0 0 -0.215 rpy=0 0 0
- added joint imu_joint: type fixed, parent base_link, child imu_link, origin xyz=-0.1464 0.0 0.26 rpy=0 0 0
- added joint lidar_l_joint: type fixed, parent base_link, child lidar_l_link, origin xyz=-0.111881 0.240 0.34432 rpy=0 0 1.57079632679
- added joint lidar_r_joint: type fixed, parent base_link, child lidar_r_link, origin xyz=-0.111881 -0.240 0.34432 rpy=0 0 -1.57079632679
- added joint zed_camera_center_joint: type fixed, parent zed_camera_link, child zed_camera_center, origin xyz=0 0 0.01325 rpy=0 0 0
- added joint zed_joint: type fixed, parent head_link2, child zed_camera_link, origin xyz=0.0238122 -0.00651797 -0.0242094 rpy=0 0 0
- added joint zed_left_camera_joint: type fixed, parent zed_camera_center, child zed_left_camera_frame, origin xyz=0 0.0315 0 rpy=0 0 0
- added joint zed_left_camera_optical_joint: type fixed, parent zed_left_camera_frame, child zed_left_camera_optical_frame, origin xyz=0 0 0 rpy=-1.57079632679 0.0 -1.57079632679
- added joint zed_right_camera_joint: type fixed, parent zed_camera_center, child zed_right_camera_frame, origin xyz=0 -0.0315 0 rpy=0 0 0
- added joint zed_right_camera_optical_joint: type fixed, parent zed_right_camera_frame, child zed_right_camera_optical_frame, origin xyz=0 0 0 rpy=-1.57079632679 0.0 -1.57079632679
- joint arm_l_joint7: limit lower=-1.8201 upper=1.5804 effort=1000 velocity=4.8 -> lower=-1.5804 upper=1.8201 effort=1000 velocity=4.8
- joint arm_r_joint7: limit lower=-1.5804 upper=1.8201 effort=1000 velocity=4.8 -> lower=-1.8201 upper=1.5804 effort=1000 velocity=4.8
- joint head_joint1: origin xyz=0.0494878 0 0.102123 rpy=0 0 0 -> xyz=0.049483 0 0.102130 rpy=0 0 0
- joint head_joint2: origin xyz=0.0365694 0 0.0563797 rpy=0 0 0 -> xyz=0.040 0 0.054 rpy=0 0 0

File: resources/ffw_sg2/ffw_sg2_spherized_approx.urdf (robot description, URDF)
Before this commit: robot ffw_sg2_follower, 40 links, 39 joints
Links:
- removed link camera_l_bottom_screw_frame
- removed link camera_l_link
- removed link camera_r_bottom_screw_frame
- removed link camera_r_link
- removed link world
- added link camera_left_bottom_screw_frame
- added link camera_left_link
- added link camera_right_bottom_screw_frame
- added link camera_right_link
- added link end_effector_l_link
- added link end_effector_r_link
- added link imu_link
- added link lidar_l_link
- added link lidar_r_link
- added link zed_camera_center
- added link zed_camera_link
- added link zed_left_camera_frame
- added link zed_left_camera_optical_frame
- added link zed_right_camera_frame
- added link zed_right_camera_optical_frame
Joints:
- removed joint camera_l_joint
- removed joint camera_l_link_joint
- removed joint camera_r_joint
- removed joint camera_r_link_joint
- removed joint world_fixed
- added joint camera_left_joint: type fixed, parent arm_l_link7, child camera_left_bottom_screw_frame, origin xyz=0.108236 -0.021 -0.062552 rpy=-1.57079632679 1.66678943569 0
- added joint camera_left_link_joint: type fixed, parent camera_left_bottom_screw_frame, child camera_left_link, origin xyz=0.01085 0.009 0.021 rpy=0 0 0
- added joint camera_right_joint: type fixed, parent arm_r_link7, child camera_right_bottom_screw_frame, origin xyz=0.108236 -0.021 -0.062552 rpy=-1.57079632679 1.66678943569 0
- added joint camera_right_link_joint: type fixed, parent camera_right_bottom_screw_frame, child camera_right_link, origin xyz=0.01085 0.009 0.021 rpy=0 0 0
- added joint end_effector_l_joint: type fixed, parent arm_l_link7, child end_effector_l_link, origin xyz=0 0 -0.215 rpy=0 0 0
- added joint end_effector_r_joint: type fixed, parent arm_r_link7, child end_effector_r_link, origin xyz=0 0 -0.215 rpy=0 0 0
- added joint imu_joint: type fixed, parent base_link, child imu_link, origin xyz=-0.1464 0.0 0.26 rpy=0 0 0
- added joint lidar_l_joint: type fixed, parent base_link, child lidar_l_link, origin xyz=-0.111881 0.240 0.34432 rpy=0 0 1.57079632679
- added joint lidar_r_joint: type fixed, parent base_link, child lidar_r_link, origin xyz=-0.111881 -0.240 0.34432 rpy=0 0 -1.57079632679
- added joint zed_camera_center_joint: type fixed, parent zed_camera_link, child zed_camera_center, origin xyz=0 0 0.01325 rpy=0 0 0
- added joint zed_joint: type fixed, parent head_link2, child zed_camera_link, origin xyz=0.0238122 -0.00651797 -0.0242094 rpy=0 0 0
- added joint zed_left_camera_joint: type fixed, parent zed_camera_center, child zed_left_camera_frame, origin xyz=0 0.0315 0 rpy=0 0 0
- added joint zed_left_camera_optical_joint: type fixed, parent zed_left_camera_frame, child zed_left_camera_optical_frame, origin xyz=0 0 0 rpy=-1.57079632679 0.0 -1.57079632679
- added joint zed_right_camera_joint: type fixed, parent zed_camera_center, child zed_right_camera_frame, origin xyz=0 -0.0315 0 rpy=0 0 0
- added joint zed_right_camera_optical_joint: type fixed, parent zed_right_camera_frame, child zed_right_camera_optical_frame, origin xyz=0 0 0 rpy=-1.57079632679 0.0 -1.57079632679
- joint arm_l_joint7: limit lower=-1.8201 upper=1.5804 effort=1000 velocity=4.8 -> lower=-1.5804 upper=1.8201 effort=1000 velocity=4.8
- joint arm_r_joint7: limit lower=-1.5804 upper=1.8201 effort=1000 velocity=4.8 -> lower=-1.8201 upper=1.5804 effort=1000 velocity=4.8
- joint head_joint1: origin xyz=0.0494878 0 0.102123 rpy=0 0 0 -> xyz=0.049483 0 0.102130 rpy=0 0 0
- joint head_joint2: origin xyz=0.0365694 0 0.0563797 rpy=0 0 0 -> xyz=0.040 0 0.054 rpy=0 0 0
